File: MotorDriver/MotorDriver.kicad_sch (KiCad schematic)
At the start: 0 parts

Commit message: start driver
Parts:
- added C1: 0.01uF, Package_DIP:DIP-8_W7.62mm, symbol Device:C
- added C2, C3: 0.1uF, Package_DIP:DIP-8_W7.62mm, symbol Device:C
- added C4: 0.47uF, Package_DIP:DIP-8_W7.62mm, symbol Device:C
- added J1: Conn_01x06_Pin, Package_DIP:DIP-20_W7.62mm, symbol Connector:Conn_01x06_Pin
- added R1: 1M, symbol Device:R
- added R2: R_Variable, Package_SO:TSSOP-20_4.4x6.5mm_P0.65mm, symbol Device:R_Variable
- added R3: R, symbol Device:R
- added U1: DRV8825PWPR, PWP28_5P18X3P1, symbol 2026-09-06_00-32-59:DRV8825PWPR
Connections:
- new net +12V: C2.2, C3.2, J1.2 (Pin_2), R1.1, U1.11 (VMB), U1.4 (VMA)
- new net +3V3: C4.2, R2.1, U1.15 (V3P3OUT)
- new net CP1: C1.1, U1.1 (CP1)
- new net CP2: C1.2, U1.2 (CP2)
- new net Dir: J1.5 (Pin_5)
- new net GND: C3.1, C4.1, J1.1 (Pin_1), J1.3 (Pin_3), R3.2, U1.14 (GND), U1.28 (GND)
- new net Sleep: J1.6 (Pin_6)
- new net Step: J1.4 (Pin_4)
- new net VCP: C2.1, R1.2, U1.3 (VCP)
- new net VREF: R2.2, R3.1, U1.12 (AVREF), U1.13 (BVREF)

Commit message: pcb
Parts:
- removed J1: Conn_01x06_Pin, Package_DIP:DIP-20_W7.62mm, symbol Connector:Conn_01x06_Pin
- removed R2: R_Variable, Package_SO:TSSOP-20_4.4x6.5mm_P0.65mm, symbol Device:R_Variable
- added C5: 0.1uF, Capacitor_SMD:C_1206_3216Metric, symbol Device:C
- added C6: 100uF, Capacitor_THT:CP_Radial_D6.3mm_P2.50mm, symbol Device:C_Polarized
- added D1: RED LED, LED_SMD:LED_1206_3216Metric, symbol Device:LED
- added J1: Conn_01x07_Socket, Connector_PinSocket_2.54mm:PinSocket_1x07_P2.54mm_Vertical, symbol Connector:Conn_01x07_Socket
- added J2: Conn_01x04_Pin, Connector_PinHeader_2.54mm:PinHeader_1x04_P2.54mm_Vertical, symbol Connector:Conn_01x04_Pin
- added R4, R5: 200M, Resistor_SMD:R_1206_3216Metric, symbol Device:R
- added R6: 10K, Resistor_SMD:R_1206_3216Metric, symbol Device:R
- added R7: 1K, Resistor_SMD:R_1206_3216Metric, symbol Device:R
- added R8: TC33X-2-503E, footprints:TRIM_TC33X-2-503E, symbol TC33X-2-503E:TC33X-2-503E
- added S1: DS01C-254-S-03BE, footprints:SW_DS01C-254-S-03BE, symbol DS01C-254-S-03BE:DS01C-254-S-03BE
- C1, C2, C3, C4: footprint Package_DIP:DIP-8_W7.62mm -> Capacitor_SMD:C_1206_3216Metric
- R1: footprint (none) -> Resistor_SMD:R_1206_3216Metric; ID (none) -> CHV1206-FX-1004ELFTR-ND; Supplier (none) -> DigiKey
- R3: value R -> 20K; footprint (none) -> Resistor_SMD:R_1206_3216Metric; ID (none) -> RNCP1206FTD20K0; Supplier (none) -> DigiKey
Connections:
- net +12V: now also C5.2, C6.1, J1.1 (Pin_1)
- net +3V3: now also R6.1, R8.3, S1.1B, S1.2B, S1.3B
- net Dir: now also U1.20 (DIR), J1.6 (Pin_6)
- net GND: now also U1.29 (EPAD), C5.1, C6.2, D1.1 (K), J1.2 (Pin_2), J1.3 (Pin_3), R4.1, R5.1
- net Sleep: now also U1.17 (NSLEEP), J1.4 (Pin_4)
- net Step: now also U1.22 (STEP), J1.7 (Pin_7)
- net VREF: now also R8.2
- net B2: now reaches U1.10 (BOUT1)
- net B2: now also J2.4 (Pin_4)
- net Fault: now reaches U1.18 (NFAULT)
- net Fault: now also R7.1
- net Decay: now reaches U1.19 (DECAY)
- net Decay: now also J1.5 (Pin_5)
- net MODE0: now reaches U1.24 (MODE0)
- net MODE0: now also S1.3A
- net MODE1: now reaches U1.25 (MODE1)
- net MODE1: now also S1.2A
- net MODE2: now reaches U1.26 (MODE2)
- net MODE2: now also S1.1A
- net NHome: now reaches U1.27 (NHOME)
- net NHome: now also R6.2
- net A1: now reaches U1.5 (AOUT1)
- net A1: now also J2.1 (Pin_1)
- net at U1.6 (ISENA): now also R4.2
- net A2: now reaches U1.7 (AOUT2)
- net A2: now also J2.3 (Pin_3)
- net B1: now reaches U1.8 (BOUT2)
- net B1: now also J2.2 (Pin_2)
- net at U1.9 (ISENB): now also R5.2
- new net: D1.2 (A), R7.2
- no-connect marks 0 -> 4
Other:
- moved on the sheet: C1, C2, C3, R1, R3
