File: HAT/HAT.kicad_sch (KiCad schematic)
At the start: 4 parts, among them J1 RPi_GPIO, J2 GPS Module

Commit message: PUSH
Parts:
- added SW1: SW_Push, symbol Switch:SW_Push
- added SW2, SW3: SW_SPDT_XKB_DMx-xxxx-1, symbol Switch:SW_SPDT_XKB_DMx-xxxx-1
Connections:
- net +3V3: now also J1.1 (3.3V), J1.17 (3.3V)
- net GND: now also SW1.2, SW2.2 (B), SW3.2 (B)
- net RebootButton: now reaches J1.12 (BCM18_PCM_C)
- net RebootButton: now also SW1.1
- net AzimuthSwitch: now reaches J1.16 (BCM23)
- net AzimuthSwitch: now also SW2.1 (A)
- net ElevationSwitch: now reaches J1.18 (BCM24)
- net ElevationSwitch: now also SW3.1 (A)
- net +5V: now reaches J1.2 (5V)
- net +5V: now also J1.4 (5V)
- no-connect marks 0 -> 2
Other:
- added sheet PowerInput (PowerIn.kicad_sch)
- added sheet PowerRegulator (PowerReg.kicad_sch)
- moved on the sheet: J2, R5, R6

Commit message: happiness
Parts:
- added MD1, MD2: (no value), symbol MotorDriver:MotorDriver
- added R8, R9: 1k, symbol Device:R
- J1, J2, R5, R6, SW1, SW2, SW3: Supplier (none) -> DigiKey
Connections:
- net AzimuthSwitch: now also R8.1; no longer SW2.1 (A)
- net ElevationSwitch: now also R9.1; no longer SW3.1 (A)
- net GND: now also J1.30 (GND), MD1.2 (GND), MD2.2 (GND)
- net RebootButton: now also J1.8 (BCM14_TXD); no longer J1.12 (BCM18_PCM_C)
- net MD1_Detect: now reaches J1.11 (BCM17)
- net MD1_Detect: now also MD1.3 (Detect)
- net MD1_Sleep: now reaches J1.13 (BCM27)
- net MD1_Sleep: now also MD1.4 (Sleep)
- net MD1_Decay: now reaches J1.15 (BCM22)
- net MD1_Decay: now also MD1.5 (Decay)
- net MD1_Dir: now reaches J1.19 (BCM10_MOSI)
- net MD1_Dir: now also MD1.6 (Dir)
- net MD2_Detect: now reaches J1.23 (BCM11_SCLK)
- net MD2_Detect: now also MD2.3 (Detect)
- net MD2_Sleep: now reaches J1.27 (BCM0_ID_SD)
- net MD2_Sleep: now also MD2.4 (Sleep)
- net MD2_Decay: now reaches J1.29 (BCM5)
- net MD2_Decay: now also MD2.5 (Decay)
- net MD2_Dir: now reaches J1.31 (BCM6)
- net MD2_Dir: now also MD2.6 (Dir)
- net MD1_Step: now reaches J1.35 (BCM19_MISO_PCM_FS)
- net MD1_Step: now also MD1.7 (Step)
- new net: R8.2, SW2.1 (A)
- new net: R9.2, SW3.1 (A)
- new net +12V: MD1.1 (+12V), MD2.1 (+12V)
- new net MD2_Step: J1.12 (BCM18_PCM_C), MD2.7 (Step)
- no-connect marks 2 -> 13
Other:
- note added: "12v -> 5v Power Reg"
- note added: "12v Input"
- note added: "BNO055 Accel/Gyro/Magno"
- note added: "GPS Module Connector"
- note added: "Motor Driver Connection"
- note added: "Motor Limit Switches"
- note added: "Notes - Not all parts have been chosen yet so some have been left blank."
- note added: "Parts R5-6: RMCF1206ZT0R00 GPS: ATGM336H"
- note added: "Raspberry Pi 4 GPIO Connector"
- note added: "Reboot Button"
- company: (none) -> Grilled Cheese Engineering
- title: (none) -> Antenna Rotor Hat Main Sheet
- moved on the sheet: J1, J2, R5, R6, SW1, SW2, SW3
