File: HAT/PowerIn.kicad_sch (KiCad schematic)
At the start: 3 parts, among them J3 Screw_Terminal_01x02, J4 Barrel_Jack_MountingPin

Commit message: happiness
Parts:
- J3, J4: Supplier (none) -> DigiKey
Other:
- note added: "Notes: - Supports 2 methods of input, barrel jack and screw terminal - Fuse will trip if more than 8A is pulled through the circuit. This is well above our estimated max current draw of 6A"
- note added: "Power Input Circuit"
- moved on the sheet: F1, J3, J4
