File: HAT/PowerReg.kicad_sch (KiCad schematic)
At the start: 6 parts, among them U2 LM1085-5.0

Commit message: happiness
Parts:
- C6, C7: ID (none) -> 50YXJ10M5X11; Supplier (none) -> DigiKey
- C8, D1, R7: Supplier (none) -> DigiKey
- U2: ID (none) -> LM1085IT-5.0/NOPB-ND; Supplier (none) -> DigiKey
Other:
- note added: "12v to 5v Power Regulator"
- note added: "Parts: - U2: LM1085IT-5.0/NOPB - C6-7: 50YXJ10M5X11 - C8: CL21B104KBCNNNC - R7: CR1206-FX-1001ELF - D1: LTST-C150KRKT"
Changed lines of the file:
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@@
 	(generator_version "10.0")
 	(paper "A4")
+	(title_block
+		(date "2026-09-06")
+		(rev "0.1.0")
+		(comment 1 "Main HAT PCB Designed by Josh Carlson")
+		(comment 2 "Motor Driver by Lucas Moidel")
+	)
+	(rectangle
+		(start 81.28 39.37)
+		(end 251.46 127)
+		(stroke
+			(width 0.508)
+			(type solid)
+		)
+		(fill
+			(type none)
+		)
+	)
+	(text "12v to 5v Power Regulator"
+		(exclude_from_sim no)
+		(at 109.22 46.482 0)
+		(effects
+			(font
+				(size 2.286 2.286)
+				(thickness 0.4572)
+				(bold yes)
+			)
+		)
+	)
+	(text "Parts:\n- U2: LM1085IT-5.0/NOPB\n- C6-7: 50YXJ10M5X11\n- C8: CL21B104KBCNNNC\n- R7: CR1206-FX-1001ELF\n- D1: LTST-C150KRKT"
+		(exclude_from_sim no)
+		(at 212.09 94.488 0)
+		(effects
+			(font
+				(size 1.27 1.27)
+			)
+			(justify left)
+		)
+	)
 	(junction
 		(at 162.56 92.71)
@@
 	(wire
 		(pts
-			(xy 106.68 80.01) (xy 130.81 80.01)
+			(xy 93.98 80.01) (xy 130.81 80.01)
 		)
 		(stroke
@@
 	(symbol
 		(lib_id "power:+12V")
-		(at 106.68 80.01 90)
+		(at 93.98 80.01 90)
 		(unit 1)
 		(body_style 1)
@@
 		(fields_autoplaced yes)
 		(property "Reference" "#PWR015"
-			(at 110.49 80.01 0)
+			(at 97.79 80.01 0)
 			(hide yes)
 			(show_name no)
@@
 		)
 		(property "Value" "+12V"
-			(at 102.87 80.0099 90)
+			(at 90.17 80.0099 90)
 			(show_name no)
 			(do_not_autoplace no)
@@
 		)
 		(property "Footprint" ""
-			(at 106.68 80.01 0)
+			(at 93.98 80.01 0)
 			(hide yes)
 			(show_name no)
@@
 		)
 		(property "Datasheet" ""
-			(at 106.68 80.01 0)
+			(at 93.98 80.01 0)
 			(hide yes)
 			(show_name no)
@@
 		)
 		(property "Description" "Power symbol creates a global label with name \"+12V\""
-			(at 106.68 80.01 0)
+			(at 93.98 80.01 0)
 			(hide yes)
 			(show_name no)
@@
 			)
 		)
+		(property "Supplier" "DigiKey"
+			(at 185.42 68.58 90)
+			(hide yes)
+			(show_name no)
+			(do_not_autoplace no)
+			(effects
+				(font
+					(size 1.27 1.27)
+				)
+			)
+		)
 		(pin "1"
 		)
@@
 			)
 		)
+		(property "Supplier" "DigiKey"
+			(at 198.12 68.58 0)
+			(hide yes)
+			(show_name no)
+			(do_not_autoplace no)
+			(effects
+				(font
+					(size 1.27 1.27)
+				)
+			)
+		)
 		(pin "2"
 		)
@@
 			)
 		)
+		(property "Supplier" "DigiKey"
+			(at 130.81 83.82 0)
+			(hide yes)
+			(show_name no)
+			(do_not_autoplace no)
+			(effects
+				(font
+					(size 1.27 1.27)
+				)
+			)
+		)
+		(property "ID" "50YXJ10M5X11"
+			(at 130.81 83.82 0)
+			(hide yes)
+			(show_name no)
+			(do_not_autoplace no)
+			(effects
+				(font
+					(size 1.27 1.27)
+				)
+			)
+		)
 		(pin "2"
 		)
@@
 			)
 		)
+		(property "Supplier" "DigiKey"
+			(at 175.26 83.82 0)
+			(hide yes)
+			(show_name no)
+			(do_not_autoplace no)
+			(effects
+				(font
+					(size 1.27 1.27)
+				)
+			)
+		)
 		(pin "1"
 		)
@@
 			)
 		)
+		(property "Supplier" "DigiKey"
+			(at 162.56 83.82 0)
+			(hide yes)
+			(show_name no)
+			(do_not_autoplace no)
+			(effects
+				(font
+					(size 1.27 1.27)
+				)
+			)
+		)
+		(property "ID" "50YXJ10M5X11"
+			(at 162.56 83.82 0)
+			(hide yes)
+			(show_name no)
+			(do_not_autoplace no)
+			(effects
+				(font
+					(size 1.27 1.27)
+				)
+			)
+		)
 		(pin "2"
 		)
@@
 			(at 147.32 80.01 0)
 			(hide yes)
+			(show_name no)
+			(do_not_autoplace no)
+			(effects
+				(font
+					(size 1.27 1.27)
+				)
+			)
+		)
+		(property "Supplier" "DigiKey"
+			(at 147.32 80.01 0)
+			(hide yes)
+			(show_name no)
+			(do_not_autoplace no)
+			(effects
+				(font
+					(size 1.27 1.27)
+				)
+			)
+		)
+		(property "ID" "LM1085IT-5.0/NOPB-ND"
+			(at 147.32 80.01 0)
+			(hide yes)
