File: HAT/magnetometer.kicad_sch (KiCad schematic)
At the start: 4 parts, among them J1 RPi_GPIO, J2 GPS Module

Commit message: First commit for the hat pcb
Parts:
- removed J1: RPi_GPIO, symbol RPiHat:RPi_GPIO
- removed J2: GPS Module, symbol Connector:Conn_01x05_Pin
- removed R5, R6: 0, symbol Device:R
- added C1: 120nF, symbol Device:C
- added C2: 1uF, symbol Device:C
- added C3: 100nF, symbol Device:C
- added C4, C5: 22pF, symbol Device:C
- added R1, R2: 10k, symbol Device:R
- added R3, R4: 0, symbol Device:R
- added U1: BNO055, Package_LGA:LGA-28_5.2x3.8mm_P0.5mm, symbol Sensor_Motion:BNO055
- added Y1: 32.768kHz, symbol Device:Crystal
Connections:
- net +3V3: now also C1.1, C3.1, R1.1, R2.1, U1.28 (VDDIO), U1.3 (VDD), U1.5 (PS1)
- net GND: now also C1.2, C2.1, C3.2, C4.1, C5.1, U1.17 (COM3), U1.18 (COM2), U1.2 (GND), U1.25 (GNDIO), U1.6 (PS0)
- new net: R2.2, U1.11 (~{RESET})
- new net: R4.2, U1.19 (COM1)
- new net: R3.2, U1.20 (COM0)
- new net: C4.2, U1.26 (XOUT32), Y1.2
- new net: C5.2, U1.27 (XIN32), Y1.1
- new net: R1.2, U1.4 (~{BOOT_LOAD_PIN})
- new net: C2.2, U1.9 (CAP)
- new net RX: R4.1
- new net TX: R3.1
- no-connect marks 0 -> 2
Other:
- removed sheet Magnetometer

Commit message: happiness
Parts:
- C1, C2, C3, C4, C5, R1, R2, R3, R4, Y1: Supplier (none) -> DigiKey
- U1: ID (none) -> BNO055; Supplier (none) -> DigiKey
Other:
- note added: "12v to 5v Power Regulator"
- note added: "Parts: - BNO055: BNO055 - C1: CC0805KRX7R9BB124 - C2: CL21F105ZBFNNNG - C3: CL21B104KBCNNNC - C4-5: CL21C220JBANNNC - R1-2: RMCF1206FT10K0 - R3-4: RMCF1206ZT0R00 - Y1: AB38T-32.768KHZ"
Changed lines of the file:
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@@
 	(generator_version "10.0")
 	(paper "A4")
+	(title_block
+		(date "2026-09-06")
+		(rev "0.1.0")
+		(comment 1 "Main HAT PCB Designed by Josh Carlson")
+		(comment 2 "Motor Driver by Lucas Moidel")
+	)
+	(rectangle
+		(start 39.37 33.02)
+		(end 273.05 160.02)
+		(stroke
+			(width 0.508)
+			(type solid)
+		)
+		(fill
+			(type none)
+		)
+	)
+	(text "Parts:\n- BNO055: BNO055\n- C1: CC0805KRX7R9BB124\n- C2: CL21F105ZBFNNNG\n- C3: CL21B104KBCNNNC\n- C4-5: CL21C220JBANNNC\n- R1-2: RMCF1206FT10K0\n- R3-4: RMCF1206ZT0R00\n- Y1: AB38T-32.768KHZ"
+		(exclude_from_sim no)
+		(at 193.04 61.468 0)
+		(effects
+			(font
+				(size 1.27 1.27)
+			)
+			(justify left)
+		)
+	)
+	(text "12v to 5v Power Regulator"
+		(exclude_from_sim no)
+		(at 67.31 40.132 0)
+		(effects
+			(font
+				(size 2.286 2.286)
+				(thickness 0.4572)
+				(bold yes)
+			)
+		)
+	)
 	(junction
 		(at 116.84 59.69)
@@
 		(property "Description" "Resistor"
 			(at 92.71 78.74 0)
+			(hide yes)
+			(show_name no)
+			(do_not_autoplace no)
+			(effects
+				(font
+					(size 1.27 1.27)
+				)
+			)
+		)
+		(property "Supplier" "DigiKey"
+			(at 92.71 78.74 90)
 			(hide yes)
 			(show_name no)
@@
 			)
 		)
+		(property "Supplier" "DigiKey"
+			(at 114.3 91.44 0)
+			(hide yes)
+			(show_name no)
+			(do_not_autoplace no)
+			(effects
+				(font
+					(size 1.27 1.27)
+				)
+			)
+		)
+		(property "ID" "BNO055"
+			(at 114.3 91.44 0)
+			(hide yes)
+			(show_name no)
+			(do_not_autoplace no)
+			(effects
+				(font
+					(size 1.27 1.27)
+				)
+			)
+		)
 		(pin "13"
 		)
@@
 			)
 		)
+		(property "Supplier" "DigiKey"
+			(at 68.58 100.33 90)
+			(hide yes)
+			(show_name no)
+			(do_not_autoplace no)
+			(effects
+				(font
+					(size 1.27 1.27)
+				)
+			)
+		)
 		(pin "1"
 		)
@@
 			)
 		)
+		(property "Supplier" "DigiKey"
+			(at 170.18 91.44 90)
+			(hide yes)
+			(show_name no)
+			(do_not_autoplace no)
+			(effects
+				(font
+					(size 1.27 1.27)
+				)
+			)
+		)
 		(pin "1"
 		)
@@
 			)
 		)
+		(property "Supplier" "DigiKey"
+			(at 154.94 85.09 90)
+			(hide yes)
+			(show_name no)
+			(do_not_autoplace no)
+			(effects
+				(font
+					(size 1.27 1.27)
+				)
+			)
+		)
 		(pin "1"
 		)
@@
 			)
 		)
+		(property "Supplier" "DigiKey"
+			(at 92.71 88.9 90)
+			(hide yes)
+			(show_name no)
+			(do_not_autoplace no)
+			(effects
+				(font
+					(size 1.27 1.27)
+				)
+			)
+		)
 		(pin "1"
 		)
@@
 		(property "Description" "Unpolarized capacitor"
 			(at 107.95 66.04 0)
+			(hide yes)
+			(show_name no)
+			(do_not_autoplace no)
+			(effects
+				(font
+					(size 1.27 1.27)
+				)
+			)
+		)
+		(property "Supplier" "DigiKey"
+			(at 107.95 66.04 90)
 			(hide yes)
 			(show_name no)
@@
 			)
 		)
+		(property "Supplier" "DigiKey"
+			(at 132.08 59.69 90)
+			(hide yes)
+			(show_name no)
+			(do_not_autoplace no)
+			(effects
+				(font
+					(size 1.27 1.27)
+				)
+			)
+		)
 		(pin "1"
 		)
@@
 			)
 		)
+		(property "Supplier" "DigiKey"
+			(at 140.97 104.14 90)
+			(hide yes)
+			(show_name no)
+			(do_not_autoplace no)
+			(effects
+				(font
+					(size 1.27 1.27)
+				)
+			)
+		)
 		(pin "1"
 		)
@@
 			)
 		)
+		(property "Supplier" "DigiKey"
+			(at 68.58 106.68 90)
+			(hide yes)
+			(show_name no)
+			(do_not_autoplace no)
+			(effects
+				(font
+					(size 1.27 1.27)
+				)
+			)
+		)
 		(pin "1"
 		)
@@
 			(hide yes)
 			(show_name no)
+			(do_not_autoplace no)
+			(effects
+				(font
+					(size 1.27 1.27)
+				)
+			)
+		)
+		(property "Supplier" "DigiKey"
+			(at 170.18 78.74 90)
+			(hide yes)
+			(show_name no)
